Commit message: 修改防碰撞的路径

File: resources/mobile_manipulator/ridgeback_ur5/urdf/ridgeback_ur5.urdf (robot description, URDF)
Before this commit: robot ridgeback, 29 links, 28 joints
Links:
- link chassis_link: geometry collision mesh filename=file:///home/xiaoyu/demo01_ocs2_ws/src/ocs2_robotic_assets/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; visual mesh filename=package://ocs2_robotic_assets/resources/mobile_manipulator/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
- link top_link: geometry collision mesh filename=file:///home/xiaoyu/demo01_ocs2_ws/src/ocs2_robotic_assets/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; visual mesh filename=package://ocs2_robotic_assets/resources/mobile_manipulator/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
- link ur_arm_base_link_inertia: geometry collision mesh filename=file:///home/xiaoyu/demo01_ocs2_ws/src/ocs2_robotic_assets/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; visual mesh filename=package://ocs2_robotic_assets/resources/mobile_manipulator/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
- link ur_arm_forearm_link: geometry collision mesh filename=file:///home/xiaoyu/demo01_ocs2_ws/src/ocs2_robotic_assets/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; visual mesh filename=package://ocs2_robotic_assets/resources/mobile_manipulator/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
- link ur_arm_shoulder_link: geometry collision mesh filename=file:///home/xiaoyu/demo01_ocs2_ws/src/ocs2_robotic_assets/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; visual mesh filename=package://ocs2_robotic_assets/resources/mobile_manipulator/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
- link ur_arm_upper_arm_link: geometry collision mesh filename=file:///home/xiaoyu/demo01_ocs2_ws/src/ocs2_robotic_assets/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; visual mesh filename=package://ocs2_robotic_assets/resources/mobile_manipulator/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
- link ur_arm_wrist_1_link: geometry collision mesh filename=file:///home/xiaoyu/demo01_ocs2_ws/src/ocs2_robotic_assets/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; visual mesh filename=package://ocs2_robotic_assets/resources/mobile_manipulator/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
- link ur_arm_wrist_2_link: geometry collision mesh filename=file:///home/xiaoyu/demo01_ocs2_ws/src/ocs2_robotic_assets/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; visual mesh filename=package://ocs2_robotic_assets/resources/mobile_manipulator/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
- link ur_arm_wrist_3_link: geometry collision mesh filename=file:///home/xiaoyu/demo01_ocs2_ws/src/ocs2_robotic_assets/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; visual mesh filename=package://ocs2_robotic_assets/resources/mobile_manipulator/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
